File: modules/01. Astabil modul/astabil.brd (EAGLE design)
At the start: 44.4 x 28.9 mm, 12 parts, among them T1 BC547, T2 BC547

Commit message: Added most CAM files
Changed lines of the file:
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@@
 <?xml version="1.0" encoding="utf-8"?>
 <!DOCTYPE eagle SYSTEM "eagle.dtd">
-<eagle version="6.5.0">
+<eagle version="9.0.0">
 <drawing>
 <settings>
 <setting alwaysvectorfont="no"/>
+<setting keepoldvectorfont="yes"/>
 <setting verticaltext="up"/>
 </settings>
@@
 <param name="dpMaxLengthDifference" value="10mm"/>
 <param name="dpGapFactor" value="2.5"/>
-<param name="checkGrid" value="0"/>
 <param name="checkAngle" value="0"/>
 <param name="checkFont" value="1"/>
 <param name="checkRestrict" value="1"/>
+<param name="checkStop" value="0"/>
+<param name="checkValues" value="0"/>
 <param name="useDiameter" value="13"/>
 <param name="maxErrors" value="50"/>
@@
 <pass name="Default">
 <param name="RoutingGrid" value="50mil"/>
+<param name="AutoGrid" value="1"/>
+<param name="Efforts" value="0"/>
+<param name="TopRouterVariant" value="1"/>
 <param name="tpViaShape" value="round"/>
 <param name="PrefDir.1" value="|"/>
@@
 <element name="R3" library="resistor" package="0207/10" value="330" x="17.78" y="13.97" rot="R90"/>
 <element name="R4" library="resistor" package="0207/10" value="330" x="31.75" y="13.97" rot="R90"/>
-<element name="LED1" library="led" package="LED5MM" value="" x="17.78" y="22.86" rot="R270"/>
-<element name="LED2" library="led" package="LED5MM" value="" x="31.75" y="22.86" rot="R270"/>
+<element name="LED1" library="led" package="LED5MM" value="" x="17.78" y="22.86" smashed="yes" rot="R270">
+<attribute name="NAME" x="20.8534" y="22.225" size="1.27" layer="25" ratio="10" rot="R270"/>
+<attribute name="VALUE" x="15.9766" y="19.6596" size="1.27" layer="27" ratio="10" rot="R270"/>
+</element>
+<element name="LED2" library="led" package="LED5MM" value="" x="31.75" y="22.86" smashed="yes" rot="R270">
+<attribute name="NAME" x="27.2034" y="22.225" size="1.27" layer="25" ratio="10" rot="R270"/>
+<attribute name="VALUE" x="29.9466" y="19.6596" size="1.27" layer="27" ratio="10" rot="R270"/>
+</element>
 <element name="C1" library="resistor" package="E3,5-8" value="10u" x="25.4" y="12.7" rot="R180"/>
 <element name="C2" library="resistor" package="E3,5-8" value="10u" x="25.4" y="3.81" smashed="yes">
