File: modules/07. Erősítő modul/erősítő.brd (EAGLE design)
At the start: 57.1 x 34 mm, 17 parts, among them IC1 TDA2030V

Commit message: Added most CAM files
Parts:
- U$2: value GANZ-CONNECTOR-OUT -> (none)
Changed lines of the file:
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@@
 <?xml version="1.0" encoding="utf-8"?>
 <!DOCTYPE eagle SYSTEM "eagle.dtd">
-<eagle version="6.5.0">
+<eagle version="9.0.0">
 <drawing>
 <settings>
 <setting alwaysvectorfont="no"/>
+<setting keepoldvectorfont="yes"/>
 <setting verticaltext="up"/>
 </settings>
-<grid distance="0.05" unitdist="inch" unit="inch" style="lines" multiple="1" display="no" altdistance="0.025" altunitdist="inch" altunit="inch"/>
+<grid distance="0.025" unitdist="inch" unit="inch" style="lines" multiple="1" display="no" altdistance="0.025" altunitdist="inch" altunit="inch"/>
 <layers>
 <layer number="1" name="Top" color="4" fill="1" visible="yes" active="yes"/>
@@
 <param name="dpMaxLengthDifference" value="10mm"/>
 <param name="dpGapFactor" value="2.5"/>
-<param name="checkGrid" value="0"/>
 <param name="checkAngle" value="0"/>
 <param name="checkFont" value="1"/>
 <param name="checkRestrict" value="1"/>
+<param name="checkStop" value="0"/>
+<param name="checkValues" value="0"/>
 <param name="useDiameter" value="13"/>
 <param name="maxErrors" value="50"/>
@@
 <pass name="Default">
 <param name="RoutingGrid" value="50mil"/>
+<param name="AutoGrid" value="1"/>
+<param name="Efforts" value="0"/>
+<param name="TopRouterVariant" value="1"/>
 <param name="tpViaShape" value="round"/>
 <param name="PrefDir.1" value="|"/>
@@
 <element name="R3" library="resistor" package="0309/12" value="1R" x="45.72" y="13.97" rot="R270"/>
 <element name="R4" library="resistor" package="0309/12" value="100k" x="34.29" y="13.97" rot="R90"/>
-<element name="D1" library="diode" package="DO41-10" value="1N4004" x="49.53" y="15.24" rot="R270"/>
-<element name="D2" library="diode" package="DO41-10" value="1N4004" x="38.1" y="15.24" rot="R90"/>
-<element name="C1" library="resistor" package="C075-032X103" value="150n" x="41.91" y="12.7" rot="R90"/>
+<element name="D1" library="diode" package="DO41-10" value="1N4004" x="49.53" y="15.24" smashed="yes" rot="R270">
+<attribute name="NAME" x="51.181" y="17.272" size="1.27" layer="25" ratio="10" rot="R270"/>
+<attribute name="VALUE" x="51.816" y="18.542" size="1.27" layer="27" ratio="10" rot="R270"/>
+</element>
+<element name="D2" library="diode" package="DO41-10" value="1N4004" x="38.1" y="15.24" smashed="yes" rot="R90">
+<attribute name="NAME" x="36.449" y="13.208" size="1.27" layer="25" ratio="10" rot="R90"/>
+<attribute name="VALUE" x="34.798" y="21.336" size="1.27" layer="27" ratio="10"/>
+</element>
+<element name="C1" library="resistor" package="C075-032X103" value="150n" x="41.91" y="12.7" smashed="yes" rot="R90">
+<attribute name="NAME" x="40.005" y="7.874" size="1.27" layer="25" ratio="10" rot="R90"/>
+<attribute name="VALUE" x="42.418" y="19.304" size="1.27" layer="27" ratio="10" rot="R90"/>
+</element>
 <element name="C2" library="resistor" package="E2,5-7" value="10u" x="21.59" y="25.4"/>
-<element name="C3" library="resistor" package="E2,5-7" value="22u" x="16.51" y="5.08" rot="R180"/>
-<element name="C4" library="resistor" package="E2,5-7" value="4u7" x="16.51" y="13.97" rot="R180"/>
-<element name="C5" library="resistor" package="E2,5-7" value="22u" x="52.07" y="3.81" rot="R270"/>
-<element name="C6" library="resistor" package="E3,5-8" value="1000u" x="46.99" y="26.67"/>
+<element name="C3" library="resistor" package="E2,5-7" value="22u" x="16.51" y="5.08" smashed="yes" rot="R180">
+<attribute name="NAME" x="13.462" y="3.048" size="1.27" layer="25" ratio="10" rot="R180"/>
+<attribute name="VALUE" x="20.32" y="6.477" size="1.27" layer="27" ratio="10" rot="R270"/>
+</element>
+<element name="C4" library="resistor" package="E2,5-7" value="4u7" x="16.51" y="13.97" smashed="yes" rot="R180">
+<attribute name="NAME" x="13.462" y="11.938" size="1.27" layer="25" ratio="10" rot="R180"/>
+<attribute name="VALUE" x="17.907" y="19.05" size="1.27" layer="27" ratio="10" rot="R180"/>
+</element>
+<element name="C5" library="resistor" package="E2,5-7" value="22u" x="52.07" y="3.81" smashed="yes" rot="R270">
+<attribute name="NAME" x="54.102" y="0.762" size="1.27" layer="25" ratio="10" rot="R270"/>
+<attribute name="VALUE" x="57.785" y="1.778" size="1.27" layer="27" ratio="10" rot="R90"/>
+</element>
+<element name="C6" library="resistor" package="E3,5-8" value="1000u" x="46.99" y="26.67" smashed="yes">
+<attribute name="NAME" x="50.292" y="29.464" size="1.27" layer="25" ratio="10"/>
+<attribute name="VALUE" x="52.578" y="23.749" size="1.27" layer="27" ratio="10" rot="R90"/>
+</element>
 <element name="U$1" library="ganzlib" package="FE08W" value="GANZ-CONNECTOR" x="6.35" y="17.78"/>
-<element name="U$2" library="ganzlib" package="MA08-1W" value="GANZ-CONNECTOR-OUT" x="55.88" y="17.78"/>
+<element name="U$2" library="ganzlib" package="MA08-1W" value="" x="55.88" y="17.78"/>
 <element name="R5" library="resistor" package="0309/12" value="100k" x="30.48" y="13.97" rot="R90"/>
 <element name="R6" library="resistor" package="0309/12" value="100k" x="26.67" y="13.97" rot="R270"/>
