File: modules/07. Erősítő modul/erősítő.sch (EAGLE design)
At the start: 17 parts, among them IC1 TDA2030V

Commit message: Added modules
Other:
- note added: "Tervezö: Balázs Lajos Rajzoló: Kimmel Gábor"
- note removed: "Tervezö: Kimmel Gábor Rajzoló: Kimmel Gábor"
Changed lines of the file:
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@@
 <plain>
 <text x="157.48" y="-15.24" size="2.54" layer="94" font="vector">Elosztó modul</text>
-<text x="101.6" y="-12.7" size="2.54" layer="94" font="vector" align="top-left">Tervezö: Kimmel Gábor
+<text x="101.6" y="-12.7" size="2.54" layer="94" font="vector" align="top-left">Tervezö: Balázs Lajos
 Rajzoló: Kimmel Gábor</text>
 <text x="187.96" y="-27.94" size="2.54" layer="94" font="vector" align="top-left">v1</text>
