File: modules/08. Kapcsoló modul/kapcsoló.brd (EAGLE design)
At the start: 107.9 x 26.3 mm, 19 parts

Commit message: Added most CAM files
Parts:
- U$1: value GANZ-CONNECTOR-OUT -> (none)
Changed lines of the file:
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@@
 <?xml version="1.0" encoding="utf-8"?>
 <!DOCTYPE eagle SYSTEM "eagle.dtd">
-<eagle version="6.5.0">
+<eagle version="9.0.0">
 <drawing>
 <settings>
 <setting alwaysvectorfont="no"/>
+<setting keepoldvectorfont="yes"/>
 <setting verticaltext="up"/>
 </settings>
@@
 <param name="dpMaxLengthDifference" value="10mm"/>
 <param name="dpGapFactor" value="2.5"/>
-<param name="checkGrid" value="0"/>
 <param name="checkAngle" value="0"/>
 <param name="checkFont" value="1"/>
 <param name="checkRestrict" value="1"/>
+<param name="checkStop" value="0"/>
+<param name="checkValues" value="0"/>
 <param name="useDiameter" value="13"/>
 <param name="maxErrors" value="50"/>
@@
 <pass name="Default">
 <param name="RoutingGrid" value="50mil"/>
+<param name="AutoGrid" value="1"/>
+<param name="Efforts" value="0"/>
+<param name="TopRouterVariant" value="1"/>
 <param name="tpViaShape" value="round"/>
 <param name="PrefDir.1" value="|"/>
@@
 </autorouter>
 <elements>
-<element name="U$1" library="ganzlib" package="MA08-1W" value="GANZ-CONNECTOR-OUT" x="105.41" y="13.97"/>
+<element name="U$1" library="ganzlib" package="MA08-1W" value="" x="105.41" y="13.97"/>
 <element name="U$2" library="ganzlib" package="FE08W" value="GANZ-CONNECTOR" x="3.81" y="13.97"/>
 <element name="S1" library="SparkFun-Electromechanical" package="TACTILE-PTH" value="" x="19.05" y="7.62"/>
