File: modules/16. Dallamcsengő modul/dallamcsengő.brd (EAGLE design)
At the start: 62.2 x 21.3 mm, 11 parts, among them IC1 UM-66T, Q1 BC557, T1 BC547

Commit message: Added most CAM files
Parts:
- U$2: value GANZ-CONNECTOR-OUT -> (none)
Changed lines of the file:
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@@
 <?xml version="1.0" encoding="utf-8"?>
 <!DOCTYPE eagle SYSTEM "eagle.dtd">
-<eagle version="6.5.0">
+<eagle version="9.0.0">
 <drawing>
 <settings>
 <setting alwaysvectorfont="no"/>
+<setting keepoldvectorfont="yes"/>
 <setting verticaltext="up"/>
 </settings>
-<grid distance="0.05" unitdist="inch" unit="inch" style="lines" multiple="1" display="no" altdistance="0.025" altunitdist="inch" altunit="inch"/>
+<grid distance="0.025" unitdist="inch" unit="inch" style="lines" multiple="1" display="no" altdistance="0.025" altunitdist="inch" altunit="inch"/>
 <layers>
 <layer number="1" name="Top" color="4" fill="1" visible="yes" active="yes"/>
@@
 <param name="dpMaxLengthDifference" value="10mm"/>
 <param name="dpGapFactor" value="2.5"/>
-<param name="checkGrid" value="0"/>
 <param name="checkAngle" value="0"/>
 <param name="checkFont" value="1"/>
 <param name="checkRestrict" value="1"/>
+<param name="checkStop" value="0"/>
+<param name="checkValues" value="0"/>
 <param name="useDiameter" value="13"/>
 <param name="maxErrors" value="50"/>
@@
 <pass name="Default">
 <param name="RoutingGrid" value="50mil"/>
+<param name="AutoGrid" value="1"/>
+<param name="Efforts" value="0"/>
+<param name="TopRouterVariant" value="1"/>
 <param name="tpViaShape" value="round"/>
 <param name="PrefDir.1" value="|"/>
@@
 </autorouter>
 <elements>
-<element name="T1" library="transistor" package="TO92" value="BC547" x="29.21" y="5.08" rot="R90"/>
+<element name="T1" library="transistor" package="TO92" value="BC547" x="29.21" y="5.08" smashed="yes" rot="R90">
+<attribute name="NAME" x="28.575" y="8.255" size="1.27" layer="25" ratio="10" rot="R90"/>
+<attribute name="VALUE" x="26.035" y="0.635" size="1.27" layer="27" ratio="10"/>
+</element>
 <element name="Q1" library="transistor-pnp" package="TO92" value="BC557" x="38.1" y="5.08" rot="R90"/>
 <element name="C1" library="resistor" package="E5-8,5" value="47u" x="16.51" y="5.08" rot="R270"/>
 <element name="R1" library="resistor" package="0309/12" value="100k" x="22.86" y="10.16" rot="R270"/>
 <element name="R2" library="resistor" package="0309/12" value="10k" x="33.02" y="10.16" rot="R90"/>
-<element name="D1" library="diode" package="DO35Z10" value="ZPD3,3" x="45.72" y="10.16" rot="R270"/>
+<element name="D1" library="diode" package="DO35Z10" value="ZPD3,3" x="45.72" y="10.16" smashed="yes" rot="R270">
+<attribute name="NAME" x="46.99" y="12.446" size="1.27" layer="25" ratio="10" rot="R270"/>
+<attribute name="VALUE" x="46.99" y="17.526" size="1.27" layer="27" ratio="10" rot="R270"/>
+</element>
 <element name="R3" library="resistor" package="0309/12" value="10k" x="41.91" y="10.16" rot="R90"/>
 <element name="IC1" library="ganzlib" package="TO92-DCS" value="UM-66T" x="50.8" y="8.89" rot="R90"/>
 <element name="U$1" library="ganzlib" package="FE08W" value="GANZ-CONNECTOR" x="3.81" y="10.16"/>
-<element name="U$2" library="ganzlib" package="MA08-1W" value="GANZ-CONNECTOR-OUT" x="58.42" y="10.16"/>
+<element name="U$2" library="ganzlib" package="MA08-1W" value="" x="58.42" y="10.16"/>
 <element name="S1" library="SparkFun-Electromechanical" package="TACTILE-PTH" value="" x="27.94" y="12.7" rot="R270"/>
 </elements>
